File: templates/n64_cartridge/n64_cartridge.kicad_pcb (KiCad board)
At the start: 2 copper layers, 100 x 60 mm, 3 parts, among them J1 N64_Cartridge_Bus

Commit message: Use a sane default board setup for this template
Other:
- net class Default: clearance 0.2 -> 0.127; trace_width 0.25 -> 0.127; via_dia 0.6 -> 0.45; via_drill 0.4 -> 0.2
- net class differential routing removed
- rule trace_clearance: 0.2 -> 0.127
- rule trace_min: 0.1 -> 0.127
- rule via_min_drill: 0.3 -> 0.2
- rule via_min_size: 0.5 -> 0.45
Changed lines of the file:
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@@
   )
   (setup
-    (last_trace_width 0.25)
+    (last_trace_width 0.127)
+    (user_trace_width 0.127)
     (user_trace_width 0.4)
-    (user_trace_width 0.6)
-    (user_trace_width 0.8)
-    (trace_clearance 0.2)
+    (trace_clearance 0.127)
     (zone_clearance 0.2)
     (zone_45_only no)
-    (trace_min 0.1)
-    (via_size 0.6)
-    (via_drill 0.4)
-    (via_min_size 0.5)
-    (via_min_drill 0.3)
+    (trace_min 0.127)
+    (via_size 0.45)
+    (via_drill 0.2)
+    (via_min_size 0.45)
+    (via_min_drill 0.2)
+    (user_via 0.45 0.2)
     (uvia_size 0.3)
     (uvia_drill 0.1)
@@
   (net 33 N64_AUDIO_R)
   (net_class Default "Dies ist die voreingestellte Netzklasse."
-    (clearance 0.2)
-    (trace_width 0.25)
-    (via_dia 0.6)
-    (via_drill 0.4)
+    (clearance 0.127)
+    (trace_width 0.127)
+    (via_dia 0.45)
+    (via_drill 0.2)
     (uvia_dia 0.3)
     (uvia_drill 0.1)
@@
     (add_net "Net-(J1-Pad46)")
   )
-  (net_class "differential routing" ""
-    (clearance 0.4)
-    (trace_width 0.25)
-    (via_dia 0.6)
-    (via_drill 0.4)
-    (uvia_dia 0.3)
-    (uvia_drill 0.1)
-  )
   (module n64_cartridge:N64_Cartridge_Edge locked (layer F.Cu)
     (at 150 130)
@@
       (effects (font (size 1 1) (thickness 0.15)))
     )
+    (fp_circle (center 0 0) (end 2.5 0) (layer Cmts.User) (width 0.15))
     (fp_circle (center 0 0) (end 2.75 0) (layer F.CrtYd) (width 0.05))
-    (fp_circle (center 0 0) (end 2.5 0) (layer Cmts.User) (width 0.15))
     (fp_text user %R (at 0.3 0) (layer F.Fab) hide
       (effects (font (size 1 1) (thickness 0.15)))
@@
       (effects (font (size 1 1) (thickness 0.15)))
     )
+    (fp_circle (center 0 0) (end 2.75 0) (layer F.CrtYd) (width 0.05))
     (fp_circle (center 0 0) (end 2.5 0) (layer Cmts.User) (width 0.15))
-    (fp_circle (center 0 0) (end 2.75 0) (layer F.CrtYd) (width 0.05))
     (fp_text user %R (at 0.3 0) (layer F.Fab) hide
       (effects (font (size 1 1) (thickness 0.15)))
